File: Boards/Ethernet/Ethernet.sch (KiCad schematic (older format))
At the start: 35 parts, among them J1 CheapBusTX24-RA, J2 WIZ_J1, J3 WIZ_J2, J4 INT, SW1 LOW ADDR, SW2 HI ADDR, U1 GAL16V8, U2 GAL16V8, U3 GAL16V8, U4 GAL16V8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

Commit message: C++ version of the PiBoard software now working
Parts:
- U5, U6: symbol 74xx:74HCT244 -> Ethernet-rescue:74HCT244-74xx
Changed lines of the file:
@@
 EESchema Schematic File Version 4
 LIBS:Ethernet-cache
-EELAYER 26 0
+EELAYER 30 0
 EELAYER END
 $Descr A3 16535 11693
@@
 ~RD
 $Comp
-L 74xx:74HCT244 U5
+L Ethernet-rescue:74HCT244-74xx U5
 U 1 1 5D9BA9AF
 P 9100 5250
@@
 	9100 6050 9100 6100
 $Comp
-L 74xx:74HCT244 U6
+L Ethernet-rescue:74HCT244-74xx U6
 U 1 1 5D9F525A
 P 10750 5250
