File: Boards/PPR Board/PPR Board.sch (KiCad schematic (older format))
At the start: 37 parts, among them J1 CheapBusTX24-RA, J2 INT, J3 RTC RST, J4 Crystal, J5 mounts, SW1 HI ADDR, SW2 LOW ADDR, U1 82C54_PLCC, U10 DS12885Q, U2 74HCT245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

Commit message: C++ version of the PiBoard software now working
Parts:
- J1: symbol PPR-Board-rescue:CheapBusTX24-RA-SamacSys_Parts-PPR-Board-rescue -> PPR-Board-rescue:CheapBusTX24-RA-SamacSys_Parts-PPR-Board-rescue-PPR-Board-rescue
- U10: symbol dallas-rtc:DS12885Q -> PPR-Board-rescue:DS12885Q-dallas-rtc
- U3: symbol 22v10:22V10-PLCC -> PPR-Board-rescue:22V10-PLCC-22v10
- U5: symbol 74xx:74HCT244 -> PPR-Board-rescue:74HCT244-74xx
- U6: symbol Interface:8259A -> PPR-Board-rescue:8259A-Interface
Changed lines of the file:
@@
 EESchema Schematic File Version 4
 LIBS:PPR Board-cache
-EELAYER 26 0
+EELAYER 30 0
 EELAYER END
 $Descr A3 16535 11693
@@
 $EndDescr
 $Comp
-L PPR-Board-rescue:CheapBusTX24-RA-SamacSys_Parts-PPR-Board-rescue J1
+L PPR-Board-rescue:CheapBusTX24-RA-SamacSys_Parts-PPR-Board-rescue-PPR-Board-rescue J1
 U 1 1 5E043769
 P 900 1000
@@
 $EndComp
 $Comp
-L Interface:8259A U6
+L PPR-Board-rescue:8259A-Interface U6
 U 1 1 5E043842
 P 8600 2350
@@
 $EndComp
 $Comp
-L dallas-rtc:DS12885Q U10
+L PPR-Board-rescue:DS12885Q-dallas-rtc U10
 U 1 1 5E04395F
 P 13200 2300
@@
 	6450 4250 6450 4300
 $Comp
-L 74xx:74HCT244 U5
+L PPR-Board-rescue:74HCT244-74xx U5
 U 1 1 5C70E57B
 P 6450 6050
@@
 NoConn ~ 8450 8000
 $Comp
-L 22v10:22V10-PLCC U3
+L PPR-Board-rescue:22V10-PLCC-22v10 U3
 U 1 1 5CB0A19B
 P 5300 8600
