File: Boards/MicroSD/MiniSys MicroSD.sch (KiCad schematic (older format))
At the start: 45 parts, among them J1 CheapBusTX24-RA, J2 PORT, J3 Micro_SD_Card_Det, J4 Micro_SD_Card_Det, J5 LED, U1 74LS32, U10 74LS123, U11 GAL16V8, U2 74LS165, U3 74LS138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

Commit message: Add MicroSD CUPL files. Still untested.
Parts:
- added J6: MISO_SR, Connector_PinHeader_2.54mm:PinHeader_2x08_P2.54mm_Vertical, symbol Connector_Generic:Conn_02x08_Odd_Even
- added J7: CTRL, Connector_PinHeader_2.54mm:PinHeader_2x08_P2.54mm_Vertical, symbol Connector_Generic:Conn_02x08_Odd_Even
- C1, C10, C11, C14, C15, C16, C17, C18, C2, C3, C4, C5, C6, C7, C8, C9: footprint (none) -> Capacitor_SMD:C_0805_2012Metric_Pad1.15x1.40mm_HandSolder
- C12, C13: footprint (none) -> Capacitor_Tantalum_SMD:CP_EIA-3528-21_Kemet-B_Pad1.50x2.35mm_HandSolder
- D1: footprint (none) -> LED_SMD:LED_0805_2012Metric_Pad1.15x1.40mm_HandSolder
- J1: footprint JAE_TX24-120R-LT-H1E -> SmacSys-Parts:JAE_TX24-120R-LT-H1E
- J2: footprint (none) -> Connector_PinHeader_2.54mm:PinHeader_2x07_P2.54mm_Vertical
- J3: value Micro_SD_Card_Det -> CF0; footprint (none) -> Connector_Card:microSD_HC_Hirose_DM3AT-SF-PEJM5
- J4: value Micro_SD_Card_Det -> CF1; footprint (none) -> Connector_Card:microSD_HC_Hirose_DM3AT-SF-PEJM5
- J5: footprint (none) -> Connector_PinHeader_2.54mm:PinHeader_1x02_P2.54mm_Horizontal
- R1, R2, R3, R4, R5, R6, R7, R8, R9: footprint (none) -> Resistor_SMD:R_0805_2012Metric_Pad1.15x1.40mm_HandSolder
- U1, U4, U8, U9: footprint (none) -> Package_SO:SOIC-14_3.9x8.7mm_P1.27mm
- U10, U2, U3, U6: footprint (none) -> Package_SO:SOIC-16_3.9x9.9mm_P1.27mm
- U11, U7: footprint (none) -> Package_LCC:PLCC-20_THT-Socket
- U5: footprint (none) -> Package_SO:SOIC-20W_7.5x12.8mm_P1.27mm
Connections:
- net labels added: S0, S1, S2, S3, S4, S5, S6, S7
- wire segments 356 -> 404
Other:
- moved on the sheet: R1, U4, U5
